File: pcb/teds-pi.kicad_pcb (KiCad board)
At the start: 6 copper layers, 85 x 56 mm, 35 parts

Commit message: add POWAH! sorta.. for now...
Parts:
- added C31: 0.1uF, Capacitor_SMD:C_0402_1005Metric, F.Cu at (152.6, 82.3)
- added J1: USB_C_Receptacle_USB2.0_16P, Connector_USB:USB_C_Receptacle_HRO_TYPE-C-31-M-12, F.Cu at (146.9, 68.5)
- added L1: 4.7uH, Inductor_SMD:L_Changjiang_FXL0630, F.Cu at (151.0, 77.2)
- added Q1: AO3401A, Package_TO_SOT_SMD:SOT-23, F.Cu at (143.6, 75.4)
- added Q2: AO3401A, Package_TO_SOT_SMD:SOT-23, F.Cu at (143.6, 79.8)
- added Q3: 2N7002, Package_TO_SOT_SMD:SOT-23, F.Cu at (143.6, 84.3)
- added R10: 10K, Resistor_SMD:R_0402_1005Metric, F.Cu at (157.2, 67.7)
- added R11: 100k, Resistor_SMD:R_0402_1005Metric, F.Cu at (157.2, 69.7)
- added R12: 10k, Resistor_SMD:R_0402_1005Metric, F.Cu at (157.2, 71.7)
- added R13: 100k, Resistor_SMD:R_0402_1005Metric, F.Cu at (160.1, 63.7)
- added R14: 44.2k, Resistor_SMD:R_0402_1005Metric, F.Cu at (160.1, 65.7)
- added R15: 6.04k, Resistor_SMD:R_0402_1005Metric, F.Cu at (160.1, 67.7)
- added R3: 49.9R, Resistor_SMD:R_0402_1005Metric, F.Cu at (154.2, 63.7)
- added R4: 49.9R, Resistor_SMD:R_0402_1005Metric, F.Cu at (154.2, 65.7)
- added R5: 49.9R, Resistor_SMD:R_0402_1005Metric, F.Cu at (154.2, 67.7)
- added R6: 49.9R, Resistor_SMD:R_0402_1005Metric, F.Cu at (154.2, 69.7)
- added R7: 4k7, Resistor_SMD:R_0402_1005Metric, F.Cu at (154.2, 71.7)
- added R8: 4k7, Resistor_SMD:R_0402_1005Metric, F.Cu at (157.2, 63.7)
- added R9: 10R, Resistor_SMD:R_0402_1005Metric, F.Cu at (157.2, 65.7)
- added U4: FUSB302BMPX, Package_DFN_QFN:WQFN-14-1EP_2.5x2.5mm_P0.5mm_EP1.45x1.45mm, F.Cu at (148.8, 83.7)
- added U5: ~, EasyEDA_Lib:SOIC-8_L5.0-W4.0-P1.27-LS6.0-BL-EP2.0, F.Cu at (159.4, 77.7)
- R1, R2: value R240 -> 240R
Connections:
- C1 pad 1: (no net) -> VCC_1V8_S3
- C1 pad 2: (no net) -> GND
- C2 pad 1: +1V8_DDR -> VCC_1V8_S3
- C3 pad 1: (no net) -> +1V1_DDR
- C9 pad 1: (no net) -> +0V6_DDR
- R1 pad 1: (no net) -> Net-(U2A-ZQ)
- R2 pad 1: (no net) -> Net-(U3A-ZQ)
- U1 pad A18: /DDR_CH1_LP4/4X_CKE0 -> /DDR_CH1_LP4/4X_CKE0_C
- U1 pad A35: unconnected-(U1C-DDR_CH1_LP4/4X_CKE0/LP5_CS0_D-PadA35) -> /DDR_CH1_LP4/4X_CKE0_D
- U1 pad AG39: unconnected-(U1F-I2S1_SDI3_M1/PDM0_SDI1_M1/I2C6_SCL_M0/UART1_CTSN_M2/PWM7_IR_M0/SPI3_MISO_M2/GPIO0_D0_d-PadAG39) -> /I2C6_SCL_M0
- U1 pad AK1: /DDR_CH0_LP4/4X_CKE0 -> /DDR_CH0_LP4/4X_CKE0_A
- U1 pad AL40: unconnected-(U1F-I2S1_SDI2_M1/PDM0_SDI0_M1/I2C6_SDA_M0/UART1_RTSN_M2/PWM6_M0/SPI0_MISO_M0/GPIO0_C7_d-PadAL40) -> /I2C6_SDA_M0
- U1 pad H2: unconnected-(U1B-DDR_CH0_LP4/4X_CKE0/LP5_CS0_B-PadH2) -> /DDR_CH0_LP4/4X_CKE0_B
- U1 pad W41: unconnected-(U1H-PMIC_SLEEP1/GPIO0_A2_d-PadW41) -> /VBUS_MCU_EN
- U2 pad J4: /DDR_CH0_LP4/4X_CKE0 -> Net-(U2A-CKE_a)
- U2 pad P4: /DDR_CH1_LP4/4X_CKE0 -> Net-(U2A-CKE_b)
- U3 pad J4: /DDR_CH0_LP4/4X_CKE0 -> Net-(U3A-CKE_a)
- U3 pad P4: /DDR_CH1_LP4/4X_CKE0 -> Net-(U3A-CKE_b)
