File: pcb/teds-pi.kicad_sch (KiCad schematic)
At the start: 35 parts

Commit message: add POWAH! sorta.. for now...
Parts:
- added C31: 0.1uF, Capacitor_SMD:C_0402_1005Metric, symbol Device:C
- added C32, C33: 220pF, symbol Device:C
- added C34, C35, C37, C40, C41: 0.1uF, symbol Device:C
- added C36: 10uF, symbol Device:C
- added C38, C39: 22uF, symbol Device:C
- added J1: USB_C_Receptacle_USB2.0_16P, Connector_USB:USB_C_Receptacle_HRO_TYPE-C-31-M-12, symbol Connector:USB_C_Receptacle_USB2.0_16P
- added L1: 4.7uH, Inductor_SMD:L_Changjiang_FXL0630, symbol Device:L
- added Q1, Q2: AO3401A, Package_TO_SOT_SMD:SOT-23, symbol Transistor_FET:AO3401A
- added Q3: 2N7002, Package_TO_SOT_SMD:SOT-23, symbol Transistor_FET:2N7002
- added R10: 10K, Resistor_SMD:R_0402_1005Metric, symbol Device:R
- added R11, R13: 100k, Resistor_SMD:R_0402_1005Metric, symbol Device:R
- added R12: 10k, Resistor_SMD:R_0402_1005Metric, symbol Device:R
- added R14: 44.2k, Resistor_SMD:R_0402_1005Metric, symbol Device:R
- added R15: 6.04k, Resistor_SMD:R_0402_1005Metric, symbol Device:R
- added R3, R4, R5, R6: 49.9R, Resistor_SMD:R_0402_1005Metric, symbol Device:R
- added R7, R8: 4k7, Resistor_SMD:R_0402_1005Metric, symbol Device:R
- added R9: 10R, Resistor_SMD:R_0402_1005Metric, symbol Device:R
- added U4: FUSB302BMPX, Package_DFN_QFN:WQFN-14-1EP_2.5x2.5mm_P0.5mm_EP1.45x1.45mm, symbol Interface_USB:FUSB302BMPX
- added U5: (no value), EasyEDA_Lib:SOIC-8_L5.0-W4.0-P1.27-LS6.0-BL-EP2.0, symbol EasyEDA_Lib:SY8205FCC
- R1, R2: value R240 -> 240R
Connections:
- net +1V8_DDR: no longer C1.1, C2.1
- net GND: now also C31.2, C32.2, C33.2, C34.2, C35.2, C36.2, C37.2, C38.2, C39.2, C40.2, J1.A1 (GND), J1.A12 (GND), J1.B1 (GND), J1.B12 (GND), J1.SH (SHIELD), Q3.2 (S), R12.2, R15.2, U4.12 (VCONN), U4.13 (VCONN), U4.15 (GND), U4.8 (GND), U4.9 (GND), U5.9 (GND)
- net DDR_CH0_LP4/4X_CKE0_B: now reaches U1.H2 (DDR_CH0_LP4/4X_CKE0/LP5_CS0_B)
- net DDR_CH0_LP4/4X_CKE0_B: now also R4.2
- net VBUS_MCU_EN: now reaches U1.W41 (PMIC_SLEEP1/GPIO0_A2_d)
- net VBUS_MCU_EN: now also Q3.1 (G), R12.1
- net I2C6_SCL_M0: now reaches U1.AG39 (I2S1_SDI3_M1/PDM0_SDI1_M1/I2C6_SCL_M0/UART1_CTSN_M2/PWM7_IR_M0/SPI3_MISO_M2/GPIO0_D0_d)
- net I2C6_SCL_M0: now also R8.2, U4.6 (SCL)
- net I2C6_SDA_M0: now reaches U1.AL40 (I2S1_SDI2_M1/PDM0_SDI0_M1/I2C6_SDA_M0/UART1_RTSN_M2/PWM6_M0/SPI0_MISO_M0/GPIO0_C7_d)
- net I2C6_SDA_M0: now also R7.2, U4.7 (SDA)
- net DDR_CH1_LP4/4X_CKE0_D: now reaches U1.A35 (DDR_CH1_LP4/4X_CKE0/LP5_CS0_D)
- net DDR_CH1_LP4/4X_CKE0_D: now also R6.2
- removed net DDR_CH0_LP4/4X_CKE0: U1.AK1 (DDR_CH0_LP4/4X_CKE0/LP5_CS0_A), U2.J4 (CKE_a), U3.J4 (CKE_a)
- removed net DDR_CH1_LP4/4X_CKE0: U1.A18 (DDR_CH1_LP4/4X_CKE0/LP5_CS0_C), U2.P4 (CKE_b), U3.P4 (CKE_b)
- new net: C40.1, U5.4 (SS)
- new net: R4.1, U2.P4 (CKE_b)
- new net: R13.2, U5.3 (EN)
- new net: R3.1, U2.J4 (CKE_a)
- new net: C32.1, J1.B5 (CC2), U4.1 (CC2), U4.14 (CC2)
- new net: R5.1, U3.J4 (CKE_a)
- new net: R6.1, U3.P4 (CKE_b)
- new net: C35.1, C41.2, L1.2, U5.2 (LX), U5.6 (VCC)
- new net: R14.1, R15.1, U5.5 (FB)
- new net: C34.1, R9.2, U4.2 (VBUS)
- new net: C41.1, U5.1 (BS)
- new net: Q1.1 (G), Q2.1 (G), Q3.3 (D), R11.2
- new net: Q1.3 (D), Q2.3 (D)
- new net: C33.1, J1.A5 (CC1), U4.10 (CC1), U4.11 (CC1)
- new net: J1.A6 (D+), J1.B6 (D+)
- new net: J1.A7 (D-), J1.B7 (D-)
- new net CC_INT_L: R10.2, U4.5 (INT_N)
- new net DDR_CH0_LP4/4X_CKE0_A: R3.2, U1.AK1 (DDR_CH0_LP4/4X_CKE0/LP5_CS0_A)
- new net DDR_CH1_LP4/4X_CKE0_C: R5.2, U1.A18 (DDR_CH1_LP4/4X_CKE0/LP5_CS0_C)
- new net VBUS_TYPEC: J1.A4 (VBUS), J1.A9 (VBUS), J1.B4 (VBUS), J1.B9 (VBUS), Q1.2 (S), R11.1, R9.1
- new net VCC_1V8_S3: C1.1, C2.1, R10.1
- new net VCC_3V3_S0: C31.1, R7.1, R8.1, U4.3 (VDD), U4.4 (VDD)
- new net VCC_SYS: C38.1, C39.1, L1.1, R14.2
- new net VCC_SYS_IN: C36.1, C37.1, Q2.2 (S), R13.1, U5.7 (VIN), U5.8 (VIN)
- no-connect marks 58 -> 62
Other:
- note added: "POWER"
- note added: "VDDQ"

Commit message: add rk806 + more POWAH!
Parts:
- added C42, C43, C46, C49, C51, C53, C54, C56, C60, C61, C62, C64, C65, C66, C68, C69, C70, C71, C72, C73, C74, C75, C76, C77, C78, C79: 22uF, symbol Device:C
- added C44, C45, C48: 100pF, symbol Device:C
- added C47, C50, C52, C57, C58: 47uF, symbol Device:C
- added C55, C59, C63, C67: 1uF, symbol Device:C
- added L10, L11, L12, L13, L14, L15, L16, L17, L8, L9: 0.47uH, EasyEDA_Lib:L0806, symbol Device:L
- added R16: 120K, Resistor_SMD:R_0402_1005Metric, symbol Device:R
- added R17, R20: 100K, Resistor_SMD:R_0402_1005Metric, symbol Device:R
- added R18, R22, R23, R24, R25: 100R, Resistor_SMD:R_0402_1005Metric, symbol Device:R
- added R19: 20K, Resistor_SMD:R_0402_1005Metric, symbol Device:R
- added R21: 0R, Resistor_SMD:R_0402_1005Metric, symbol Device:R
- added U6: (no value), EasyEDA_Lib:QFN-68_L7.0-W7.0-P0.35-BL-EP5.5, symbol EasyEDA_Lib:RK806-1_C5156483
Connections:
- net GND: now also C42.2, C43.2, C46.2, C47.2, C49.2, C50.2, C51.1, C52.1, C53.2, C54.2, C56.1, C57.1, C58.1, C60.1, C61.1, C62.1, C64.1, C65.1, C66.1, C68.1, C69.1, C70.1, C71.1, C72.1, C73.2, C74.2, C75.2, C76.2, C77.2, C78.2, C79.2, R17.2, R20.2
- net VCC_1V8_S3: now also C53.1, C54.1, L16.1, R21.2, U6.25 (VOUT10)
- net VCC_SYS: now also C73.1, C74.1, C75.1, C76.1, C77.1, C78.1, C79.1, U6.1 (VCC9), U6.20 (VCCIO), U6.22 (VCC4), U6.27 (VCC10), U6.33 (VCC2), U6.34 (VCC2), U6.43 (VCC7), U6.44 (VCC5), U6.52 (VCC1), U6.53 (VCC1), U6.59 (VCC11), U6.64 (VCC12)
- net PMIC_INT_L: now reaches U1.W42 (PMIC_INT_L/GPIO0_A7_u)
- net PMIC_INT_L: now also U6.19 (INT)
- new net: L12.1, U6.45 (SW5)
- new net: L15.2, U6.6 (SW8)
- new net: C48.2, R19.2, R20.1, U6.66 (FB9)
- new net: L14.1, U6.68 (SW9)
- new net: C44.2, R16.2, R17.1, U6.31 (FB6)
- new net: L10.1, U6.55 (SW3)
- new net: L8.1, U6.50 (SW1), U6.51 (SW1)
- new net: L11.2, U6.23 (SW4)
- new net: L13.2, U6.29 (SW6)
- new net: L17.1, U6.42 (SW7)
- new net: L16.2, U6.26 (SW10)
- new net: L9.1, U6.35 (SW2), U6.36 (SW2)
- new net PMIC_EXT_EN: U6.39 (EXT_EN)
- new net PMIC_PWRON: U6.4 (PWRON)
- new net PMIC_SPI_CLK: U6.17 (CLK/SCL)
- new net PMIC_SPI_CS0: U6.18 (CS)
- new net PMIC_SPI_MISO: U6.16 (MISO/PWRCRTL3)
- new net PMIC_SPI_MOSI: U6.15 (MOSI/SDA)
- new net VCC1V8_PMU_DDR_S3: R21.1
- new net VCC_2V0_PLDO_S3: C71.2, C72.2, L17.2, U6.41 (VOUT7)
- new net VCC_3V3_S3: C51.2, C52.2, L15.1, U6.5 (VOUT8)
- new net VDD2_DDR_S3: C42.1, C43.1, C44.1, L13.1, R16.1, U6.30 (VOUT6)
- new net VDD_CPU_LIT_S0: C59.1, C59.2, C60.2, C61.2, C62.2, L9.2, R23.1, R23.2, U6.37 (VOUT2)
- new net VDD_DDRQ_S0: C48.1, C49.1, C50.1, L14.2, R19.1, U6.67 (VOUT9)
- new net VDD_DDR_S0: C45.1, C45.2, C46.1, C47.1, L12.2, R18.1, R18.2, U6.46 (VOUT5)
- new net VDD_GPU_S0: C55.1, C55.2, C56.2, C57.2, C58.2, L8.2, R22.1, R22.2, U6.49 (VOUT1)
- new net VDD_LOGIC_S0: C63.1, C63.2, C64.2, C65.2, C66.2, L10.2, R24.1, R24.2, U6.56 (VOUT3)
- new net VDD_VDENC_S0: C67.1, C67.2, C68.2, C69.2, C70.2, L11.1, R25.1, R25.2, U6.24 (VOUT4)
- no-connect marks 62 -> 65
Other:
- note added: "Feedback from RK3588S"
